File: Hardware/LilyPad_Light_Sensor.sch (EAGLE design)
At the start: 14 parts, among them U3 ALS-PT19

Commit message: Fixes from double check
Parts:
- removed R24: 10k, SparkFun-Resistors:10KOHM-0603-1/10W-1%
- added LOGO1: OSHW-LOGOMINI, SparkFun-Aesthetics:OSHW-LOGOMINI
- added LOGO2: SFE_LOGO_FLAME.1_INCH, SparkFun-Aesthetics:SFE_LOGO_FLAME.1_INCH
- added R1: 10k, SparkFun-Resistors:10KOHM-0603-1/10W-1%
- renumbered U3 to U1
Connections:
- net D2: now also R1.2; no longer R24.2
- net GND: now also R1.1; no longer R24.1
Other:
- note added: "LilyPad concept and shapes by: L. Buechley and N. Seidle"
- note added: "v14"
- note removed: "v01"
Changed lines of the file:
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@@
 <drawing>
 <settings>
-<setting alwaysvectorfont="yes"/>
+<setting alwaysvectorfont="no"/>
 <setting verticaltext="up"/>
 </settings>
@@
 <part name="SEWTAPLS+" library="LilyPad-Wearables" deviceset="SEWTAP" device="_SMALL-2SIDE" value="PLUS"/>
 <part name="SEWTAPLSOUT" library="LilyPad-Wearables" deviceset="SEWTAP" device="_SMALL-2SIDE" value="OUT"/>
-<part name="R24" library="SparkFun-Resistors" deviceset="10KOHM" device="-0603-1/10W-1%" value="10k"/>
-<part name="U3" library="SparkFun-Sensors" deviceset="LIGHT_SENSOR" device="ALS" value="ALS-PT19"/>
+<part name="R1" library="SparkFun-Resistors" deviceset="10KOHM" device="-0603-1/10W-1%" value="10k"/>
+<part name="U1" library="SparkFun-Sensors" deviceset="LIGHT_SENSOR" device="ALS" value="ALS-PT19"/>
 <part name="P+8" library="SparkFun-PowerSymbols" deviceset="VCC" device=""/>
 <part name="GND24" library="SparkFun-PowerSymbols" deviceset="GND" device=""/>
@@
 <part name="FD3" library="SparkFun-Aesthetics" deviceset="FIDUCIAL" device="UFIDUCIAL"/>
 <part name="FD4" library="SparkFun-Aesthetics" deviceset="FIDUCIAL" device="UFIDUCIAL"/>
+<part name="LOGO1" library="SparkFun-Aesthetics" deviceset="OSHW-LOGO" device="MINI"/>
+<part name="LOGO2" library="SparkFun-Aesthetics" deviceset="SFE_LOGO_FLAME" device=".1_INCH"/>
 </parts>
 <sheets>
@@
 sew taps</text>
 <text x="99.06" y="172.72" size="5.08" layer="97">Light Sensor</text>
-<text x="171.45" y="11.43" size="2.54" layer="94">Marshall Taylor</text>
-<text x="238.252" y="7.112" size="2.54" layer="94">v01</text>
-<text x="148.59" y="7.112" size="2.54" layer="94">Revised by: Elias Santistevan</text>
+<text x="171.45" y="11.43" size="2.54" layer="94" font="vector">Marshall Taylor</text>
+<text x="238.252" y="7.112" size="2.54" layer="94" font="vector">v14</text>
+<text x="148.59" y="7.112" size="2.54" layer="94" font="vector">Revised by: Elias Santistevan</text>
 <text x="101.6" y="139.7" size="2.54" layer="97">VCC Range: 2.5V-5.5V</text>
+<text x="147.32" y="38.1" size="2.54" layer="94" font="vector">LilyPad concept and shapes by:
+L. Buechley and N. Seidle</text>
 </plain>
 <instances>
@@
 <attribute name="VALUE" x="128.778" y="105.918" size="1.778" layer="96"/>
 </instance>
-<instance part="R24" gate="G$1" x="121.92" y="93.98" rot="R90"/>
-<instance part="U3" gate="G$1" x="119.38" y="116.84" smashed="yes">
+<instance part="R1" gate="G$1" x="121.92" y="96.52" rot="R90"/>
+<instance part="U1" gate="G$1" x="119.38" y="116.84" smashed="yes">
 <attribute name="VALUE" x="124.46" y="114.935" size="1.778" layer="96"/>
 <attribute name="NAME" x="124.46" y="118.11" size="1.778" layer="95"/>
@@
 <instance part="FD3" gate="G$1" x="243.84" y="27.94"/>
 <instance part="FD4" gate="G$1" x="246.38" y="27.94"/>
+<instance part="LOGO1" gate="G$1" x="236.22" y="53.34"/>
+<instance part="LOGO2" gate="G$1" x="215.9" y="48.26"/>
 </instances>
 <busses>
@@
 <segment>
 <pinref part="SEWTAPLS-" gate="G$1" pin="1"/>
-<pinref part="R24" gate="G$1" pin="1"/>
-<wire x1="121.92" y1="88.9" x2="121.92" y2="86.36" width="0.1524" layer="91"/>
+<pinref part="R1" gate="G$1" pin="1"/>
+<wire x1="121.92" y1="91.44" x2="121.92" y2="86.36" width="0.1524" layer="91"/>
 <wire x1="121.92" y1="86.36" x2="124.46" y2="86.36" width="0.1524" layer="91"/>
 <wire x1="121.92" y1="86.36" x2="121.92" y2="83.82" width="0.1524" layer="91"/>
@@
 <segment>
 <pinref part="SEWTAPLS+" gate="G$1" pin="1"/>
-<pinref part="U3" gate="G$1" pin="C1"/>
+<pinref part="U1" gate="G$1" pin="C1"/>
 <wire x1="121.92" y1="121.92" x2="121.92" y2="124.46" width="0.1524" layer="91"/>
 <wire x1="121.92" y1="124.46" x2="124.46" y2="124.46" width="0.1524" layer="91"/>
@@
 <net name="D2" class="0">
 <segment>
-<wire x1="121.92" y1="99.06" x2="121.92" y2="101.6" width="0.1524" layer="91"/>
 <wire x1="121.92" y1="101.6" x2="121.92" y2="106.68" width="0.1524" layer="91"/>
 <pinref part="SEWTAPLSOUT" gate="G$1" pin="1"/>
-<pinref part="R24" gate="G$1" pin="2"/>
-<pinref part="U3" gate="G$1" pin="E1"/>
+<pinref part="R1" gate="G$1" pin="2"/>
+<pinref part="U1" gate="G$1" pin="E1"/>
 <wire x1="121.92" y1="106.68" x2="121.92" y2="111.76" width="0.1524" layer="91"/>
-<junction x="121.92" y="101.6"/>
 <wire x1="124.46" y1="106.68" x2="121.92" y2="106.68" width="0.1524" layer="91"/>
 <junction x="121.92" y="106.68"/>
-<wire x1="121.92" y1="101.6" x2="127" y2="101.6" width="0.1524" layer="91"/>
-<label x="127" y="101.6" size="1.27" layer="95" xref="yes"/>
 </segment>
 </net>

Commit message: Double Check changes!
Other:
- note added: "v20"
- note removed: "v14"
Changed lines of the file:
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@@
 <sheet>
 <plain>
-<text x="114.3" y="66.04" size="1.778" layer="97">Un-used
+<text x="114.3" y="66.04" size="1.778" layer="97" font="vector">Un-used
 sew taps</text>
-<text x="99.06" y="172.72" size="5.08" layer="97">Light Sensor</text>
+<text x="99.06" y="172.72" size="5.08" layer="97" font="vector">Light Sensor</text>
 <text x="171.45" y="11.43" size="2.54" layer="94" font="vector">Marshall Taylor</text>
-<text x="238.252" y="7.112" size="2.54" layer="94" font="vector">v14</text>
+<text x="238.252" y="7.112" size="2.54" layer="94" font="vector">v20</text>
 <text x="148.59" y="7.112" size="2.54" layer="94" font="vector">Revised by: Elias Santistevan</text>
-<text x="101.6" y="139.7" size="2.54" layer="97">VCC Range: 2.5V-5.5V</text>
+<text x="104.14" y="139.7" size="2.54" layer="97" font="vector">VCC Range: 2.5V-5.5V</text>
 <text x="147.32" y="38.1" size="2.54" layer="94" font="vector">LilyPad concept and shapes by:
 L. Buechley and N. Seidle</text>
@@
 <instance part="ST1" gate="G$1" x="132.08" y="71.12" smashed="yes"/>
 <instance part="SEWTAPLS-" gate="G$1" x="127" y="86.36" smashed="yes">
-<attribute name="VALUE" x="129.032" y="85.598" size="1.778" layer="96"/>
+<attribute name="VALUE" x="129.032" y="85.598" size="1.778" layer="96" font="vector"/>
 </instance>
 <instance part="SEWTAPLS+" gate="G$1" x="127" y="124.46" smashed="yes">
-<attribute name="VALUE" x="129.032" y="123.698" size="1.778" layer="96"/>
+<attribute name="VALUE" x="129.032" y="123.698" size="1.778" layer="96" font="vector"/>
 </instance>
 <instance part="SEWTAPLSOUT" gate="G$1" x="127" y="106.68" smashed="yes">
-<attribute name="VALUE" x="128.778" y="105.918" size="1.778" layer="96"/>
+<attribute name="VALUE" x="128.778" y="105.918" size="1.778" layer="96" font="vector"/>
 </instance>
 <instance part="R1" gate="G$1" x="121.92" y="96.52" rot="R90"/>
 <instance part="U1" gate="G$1" x="119.38" y="116.84" smashed="yes">
-<attribute name="VALUE" x="124.46" y="114.935" size="1.778" layer="96"/>
-<attribute name="NAME" x="124.46" y="118.11" size="1.778" layer="95"/>
+<attribute name="VALUE" x="124.46" y="114.935" size="1.778" layer="96" font="vector"/>
+<attribute name="NAME" x="124.46" y="118.11" size="1.778" layer="95" font="vector"/>
 </instance>
 <instance part="P+8" gate="G$1" x="121.92" y="127"/>
@@
 <instance part="FD3" gate="G$1" x="243.84" y="27.94"/>
 <instance part="FD4" gate="G$1" x="246.38" y="27.94"/>
-<instance part="LOGO1" gate="G$1" x="236.22" y="53.34"/>
+<instance part="LOGO1" gate="G$1" x="236.22" y="55.88"/>
 <instance part="LOGO2" gate="G$1" x="215.9" y="48.26"/>
 </instances>
